Commit message: CHANGES

File: src/asitlorbot8_description/urdf/imu.xacro (robot description, xacro)
@@ -5,5 +5,5 @@
         <parent link="base_link"/>
         <child link="imu_link"/>
-        <origin xyz="0 0 0.14"/>
+        <origin xyz="0.07 0 0.14"/>
     </joint>
     <link name="imu_link">
@@ -32,5 +32,5 @@
         <sensor name="imu" type="imu">
             <always_on>true</always_on>
-            <update_rate>0.1</update_rate>
+            <update_rate>100</update_rate>
             <visualize>true</visualize>
             <imu>
@@ -39,5 +39,5 @@
                         <noise type="gaussian">
                             <mean>0.0</mean>
-                            <stddev>2e-3</stddev>
+                            <stddev>2e-4</stddev>
                         </noise>
                     </x>
@@ -45,5 +45,5 @@
                         <noise type="gaussian">
                             <mean>0.0</mean>
-                            <stddev>2e-3</stddev>
+                            <stddev>2e-4</stddev>
                         </noise>
                     </y>
@@ -51,5 +51,5 @@
                         <noise type="gaussian">
                             <mean>0.0</mean>
-                            <stddev>2e-1</stddev>
+                            <stddev>2e-4</stddev>
                         </noise>
                     </z>

File: src/asitlorbot8_description/urdf/robot_core.xacro (robot description, xacro)
@@ -25,5 +25,5 @@
         <parent link="base_link"/>
         <child link="base_footprint"/>
-        <origin xyz="0 0 0" rpy="0 0 0"/>
+        <origin xyz="0 0 -0.055" rpy="0 0 0"/>
     </joint>
     <link name="base_footprint">
@@ -33,5 +33,5 @@
         <parent link="base_link"/>
         <child link="chassis"/>
-        <origin xyz="-0.06 0 0"/>
+        <origin xyz="-0.1275 0 0"/>
     </joint>
     <link name="chassis">
@@ -62,5 +62,5 @@
         <parent link="base_link"/>
         <child link="left_back_wheel"/>
-        <origin xyz="0 0.1 0" rpy="-${pi/2} 0 0" />
+        <origin xyz="0.0625 0.1 0" rpy="-${pi/2} 0 0" />
         <axis xyz="0 0 1"/>
         <!-- <limit effort="10000" velocity="1000"/> -->
@@ -109,5 +109,5 @@
         <parent link="base_link"/>
         <child link="left_front_wheel"/>
-        <origin xyz="0.125 0.1 0" rpy="-${pi/2} 0 0" />
+        <origin xyz="-0.0625 0.1 0" rpy="-${pi/2} 0 0" />
         <axis xyz="0 0 1"/>
         <!-- <limit effort="10000" velocity="1000"/> -->
@@ -156,5 +156,5 @@
         <parent link="base_link"/>
         <child link="right_back_wheel"/>
-        <origin xyz="0 -0.1 0" rpy="${pi/2} 0 0" />
+        <origin xyz="0.0625 -0.1 0" rpy="${pi/2} 0 0" />
         <axis xyz="0 0 -1"/>
         <!-- <limit effort="10000" velocity="1000"/> -->
@@ -203,5 +203,5 @@
         <parent link="base_link"/>
         <child link="right_front_wheel"/>
-        <origin xyz="0.125 -0.1 0" rpy="${pi/2} 0 0" />
+        <origin xyz="-0.0625 -0.1 0" rpy="${pi/2} 0 0" />
         <axis xyz="0 0 -1"/>
         <!-- <limit effort="10000" velocity="1000"/> -->

File: src/asitlorbot8_description/urdf/transmission.xacro (robot description, xacro)
@@ -10,5 +10,5 @@
             <hardwareInterface>hardware_interface/EffortJointInterface</hardwareInterface>
             <!-- 1 DEGREE OF ROTATION OF MOTOR CORRESPONDS TO 1 DEGREE OF ROTATION OF WHEEL -->
-            <mechanicalReduction>1.0</mechanicalReduction>
+            <mechanicalReduction>1</mechanicalReduction>
         </actuator>
     </transmission>
@@ -20,5 +20,5 @@
         <actuator name="joint_front_right_actr">
             <hardwareInterface>hardware_interface/EffortJointInterface</hardwareInterface>
-            <mechanicalReduction>1.0</mechanicalReduction>
+            <mechanicalReduction>1</mechanicalReduction>
         </actuator>
     </transmission>
