Commit message: NEW UPLOAD

File: src/asitlorbot8_description/urdf/asitlorbot8.urdf.xacro (robot description, xacro)
@@ -1,5 +1,5 @@
 <?xml version="1.0"?>
 <robot xmlns:xacro="http://www.ros.org/wiki/xacro"  name="asitlorbot8">
-    <xacro:arg name="is_sim" default="false"/>
+    <xacro:arg name="is_sim" default="true"/>
     <!-- ROBOT DESCRIPTION - LINKS AND JOINTS -->
     <xacro:include filename="robot_core.xacro"/>

File: src/asitlorbot8_description/urdf/lidar.xacro (robot description, xacro)
@@ -26,5 +26,5 @@
         <sensor name="laser" type="ray">
             <pose> 0 0 0 0 0 0 </pose>
-            <visualize>true</visualize>
+            <visualize>false</visualize>
             <update_rate>10</update_rate>
             <ray>

File: src/asitlorbot8_description/urdf/ros2_control.xacro (robot description, xacro)
@@ -11,9 +11,9 @@
             <hardware>
                 <plugin>asitlorbot8_firmware/asitlorbotInterface</plugin>
-                <param name="port">/dev/ttyUSB0</param>
+                <param name="port">/dev/ttyAMA0</param>
                 <!-- <param name="port">/dev/ttyUSB1</param> -->
             </hardware>
         </xacro:unless>
-        <!-- <joint name="left_back_wheel_hinge">
+        <joint name="left_back_wheel_hinge">
             <command_interface name="velocity">
                 <param name="min">-10</param>
@@ -30,5 +30,5 @@
             <state_interface name="velocity"/>
             <state_interface name="position"/>
-        </joint> -->
+        </joint>
         <joint name="left_front_wheel_hinge">
             <command_interface name="velocity">

Commit message: NEW UPLOAD

File: src/asitlorbot8_description/urdf/asitlorbot8.urdf.xacro (robot description, xacro)
@@ -1,5 +1,5 @@
 <?xml version="1.0"?>
 <robot xmlns:xacro="http://www.ros.org/wiki/xacro"  name="asitlorbot8">
-    <xacro:arg name="is_sim" default="true"/>
+    <xacro:arg name="is_sim" default="false"/>
     <!-- ROBOT DESCRIPTION - LINKS AND JOINTS -->
     <xacro:include filename="robot_core.xacro"/>

File: src/asitlorbot8_description/urdf/imu.xacro (robot description, xacro)
@@ -32,5 +32,5 @@
         <sensor name="imu" type="imu">
             <always_on>true</always_on>
-            <update_rate>100</update_rate>
+            <update_rate>1</update_rate>
             <visualize>true</visualize>
             <imu>

File: src/asitlorbot8_description/urdf/robot_core.xacro (robot description, xacro)
@@ -1,5 +1,5 @@
 <?xml version="1.0"?>
 <robot xmlns:xacro="http://www.ros.org/wiki/xacro"  name="asitlorbot8">
-    <xacro:arg name="is_sim" default="true"/>
+    <xacro:arg name="is_sim" default="false"/>
     <xacro:include filename="inertial_macros.xacro"/>
     <material name="white">
@@ -19,13 +19,13 @@
     </material>
     <!-- BASE LINK -->
-    <link name="base_link">
+    <link name="base_footprint">
     </link>
     <!-- BASE_FOOTPRINT LINK -->
     <joint name="base_footprint_joint" type="fixed">
-        <parent link="base_link"/>
-        <child link="base_footprint"/>
-        <origin xyz="0 0 -0.055" rpy="0 0 0"/>
-    </joint>
-    <link name="base_footprint">
+        <parent link="base_footprint"/>
+        <child link="base_link"/>
+        <origin xyz="0 0 0.055" rpy="0 0 0"/>
+    </joint>
+    <link name="base_link">
     </link>
     <!-- CHASSIS LINK -->
@@ -64,6 +64,7 @@
         <origin xyz="0.0625 0.1 0" rpy="-${pi/2} 0 0" />
         <axis xyz="0 0 1"/>
-        <!-- <limit effort="10000" velocity="1000"/> -->
-        <!-- <dynamics damping="0.7" friction="100"/> -->
+        <limit effort="10000.0" velocity="20.0" />
+        <dynamics damping="0"/>
+        <joint_properties friction="0.0" />
     </joint>
     <link name="left_back_wheel">
@@ -80,12 +81,11 @@
             <surface>
                 <friction>
-                    <fdir1>1 0 0</fdir1>
-                    <!-- <kp>50000.0</kp> -->
-                    <!-- kp and kd for rubber -->
-                    <!-- <kd>0.8</kd> -->
-                    <!-- <mu1>100</mu1> -->
-                    <!-- <mu2>100</mu2> -->
-                    <slip1>0.0</slip1>
-                    <slip2>0.0</slip2>
+                    <ode>
+                        <mu>10.0</mu>          <!-- Moderate grip in the primary direction -->
+                        <mu2>10.0</mu2>        <!-- Moderate grip in the secondary direction -->
+                        <fdir1>1 0 0</fdir1>  <!-- Aligns primary friction with the x-axis (forward direction) -->
+                        <slip1>0.0</slip1>   <!-- Small slip value for slight sliding capability -->
+                        <slip2>0.0</slip2>   <!-- Small slip value for slight sliding capability -->
+                    </ode>
                 </friction>
             </surface>
@@ -97,11 +97,13 @@
     <gazebo reference="left_back_wheel">
         <material>Gazebo/Blue</material>
-        <!-- <kp>50000.0</kp>  -->
-        <!-- kp and kd for rubber -->
-        <!-- <kd>0.8</kd> -->
-        <mu1>1</mu1>
-        <mu2>1</mu2>
-        <maxVel>0.0</maxVel>
-        <minDepth>0.00005</minDepth>
+        <mu1>1.0</mu1>
+        <mu2>1.0</mu2>
+        <kp>1000000000000.0</kp>
+        <kd>10.0</kd>
+        <minDepth>0.0001</minDepth>
+        <maxVel>0.0</maxVel>
+        <fdir1>1 0 0</fdir1>
+        <slip1>0.0</slip1>   <!-- Small slip value for slight sliding capability -->
+        <slip2>0.0</slip2>
     </gazebo>
     <!-- LEFT FRONT WHEEL LINK -->
@@ -111,6 +113,7 @@
         <origin xyz="-0.0625 0.1 0" rpy="-${pi/2} 0 0" />
         <axis xyz="0 0 1"/>
-        <!-- <limit effort="10000" velocity="1000"/> -->
-        <!-- <dynamics damping="0.7" friction="100"/> -->
+        <limit effort="10000.0" velocity="20.0" />
+        <dynamics damping="0"/>
+        <joint_properties friction="0.0" />
     </joint>
     <link name="left_front_wheel">
@@ -127,12 +130,11 @@
             <surface>
                 <friction>
-                    <fdir1>1 0 0</fdir1>
-                    <!-- <kp>50000.0</kp> -->
-                    <!-- kp and kd for rubber -->
-                    <!-- <kd>0.8</kd> -->
-                    <!-- <mu1>100</mu1>
-                    <mu2>100</mu2> -->
-                    <slip1>0.0</slip1>
-                    <slip2>0.0</slip2>
+                    <ode>
+                        <mu>1.0</mu>          <!-- Moderate grip in the primary direction -->
+                        <mu2>1.0</mu2>        <!-- Moderate grip in the secondary direction -->
+                        <fdir1>1 0 0</fdir1>  <!-- Aligns primary friction with the x-axis (forward direction) -->
+                        <slip1>0.0</slip1>   <!-- Small slip value for slight sliding capability -->
+                        <slip2>0.0</slip2>   <!-- Small slip value for slight sliding capability -->
+                    </ode>
                 </friction>
             </surface>
@@ -144,11 +146,13 @@
     <gazebo reference="left_front_wheel">
         <material>Gazebo/Blue</material>
-        <!-- <kp>50000.0</kp>  -->
-        <!-- kp and kd for rubber -->
-        <!-- <kd>0.8</kd> -->
-        <mu1>1</mu1>
-        <mu2>1</mu2>
-        <maxVel>0.0</maxVel>
-        <minDepth>0.00005</minDepth>
+        <mu1>1.0</mu1>
+        <mu2>1.0</mu2>
+        <kp>1000000000000.0</kp>
+        <kd>10.0</kd>
+        <minDepth>0.0001</minDepth>
+        <maxVel>0.0</maxVel>
+        <fdir1>1 0 0</fdir1>
+        <slip1>0.0</slip1>   <!-- Small slip value for slight sliding capability -->
+        <slip2>0.0</slip2>
     </gazebo>
     <!-- RIGHT BACK WHEEL -->
@@ -158,6 +162,7 @@
         <origin xyz="0.0625 -0.1 0" rpy="${pi/2} 0 0" />
         <axis xyz="0 0 -1"/>
-        <!-- <limit effort="10000" velocity="1000"/> -->
-        <!-- <dynamics damping="0.7" friction="100"/> -->
+        <limit effort="10000.0" velocity="20.0" />
+        <dynamics damping="0"/>
+        <joint_properties friction="0.0" />
     </joint>
     <link name="right_back_wheel">
@@ -174,12 +179,11 @@
             <surface>
                 <friction>
-                    <fdir1>1 0 0</fdir1>
-                    <!-- <kp>50000.0</kp>  -->
-                    <!-- kp and kd for rubber -->
-                    <!-- <kd>0.8</kd> -->
-                    <!-- <mu1>100</mu1>
-                    <mu2>100</mu2> -->
-                    <slip1>0.0</slip1>
-                    <slip2>0.0</slip2>
+                    <ode>
+                        <mu>1.0</mu>          <!-- Moderate grip in the primary direction -->
+                        <mu2>1.0</mu2>        <!-- Moderate grip in the secondary direction -->
+                        <fdir1>1 0 0</fdir1>  <!-- Aligns primary friction with the x-axis (forward direction) -->
+                        <slip1>0.0</slip1>   <!-- Small slip value for slight sliding capability -->
+                        <slip2>0.0</slip2>   <!-- Small slip value for slight sliding capability -->
+                    </ode>
                 </friction>
             </surface>
@@ -191,11 +195,13 @@
     <gazebo reference="right_back_wheel">
         <material>Gazebo/Blue</material>
-        <!-- <kp>50000.0</kp>  -->
-        <!-- kp and kd for rubber -->
-        <!-- <kd>0.8</kd> -->
-        <mu1>1</mu1>
-        <mu2>1</mu2>
-        <maxVel>0.0</maxVel>
-        <minDepth>0.00005</minDepth>
+        <mu1>1.0</mu1>
+        <mu2>1.0</mu2>
+        <kp>1000000000000.0</kp>
+        <kd>10.0</kd>
+        <minDepth>0.0001</minDepth>
+        <maxVel>0.0</maxVel>
+        <fdir1>1 0 0</fdir1>
+        <slip1>0.0</slip1>   <!-- Small slip value for slight sliding capability -->
+        <slip2>0.0</slip2>
     </gazebo>
     <!-- RIGHT FRONT WHEEL -->
@@ -205,6 +211,7 @@
         <origin xyz="-0.0625 -0.1 0" rpy="${pi/2} 0 0" />
         <axis xyz="0 0 -1"/>
-        <!-- <limit effort="10000" velocity="1000"/> -->
-        <!-- <dynamics damping="0.7" friction="100"/> -->
+        <limit effort="10000.0" velocity="20.0" />
+        <dynamics damping="0"/>
+        <joint_properties friction="0.0" />
     </joint>
     <link name="right_front_wheel">
@@ -221,12 +228,11 @@
             <surface>
                 <friction>
-                    <fdir1>1 0 0</fdir1>
-                    <!-- <kp>50000.0</kp>  -->
-                    <!-- kp and kd for rubber -->
-                    <!-- <kd>0.8</kd> -->
-                    <!-- <mu1>100</mu1>
-                    <mu2>100</mu2> -->
-                    <slip1>0.0</slip1>
-                    <slip2>0.0</slip2>
+                    <ode>
+                        <mu>1.0</mu>          <!-- Moderate grip in the primary direction -->
+                        <mu2>1.0</mu2>        <!-- Moderate grip in the secondary direction -->
+                        <fdir1>1 0 0</fdir1>  <!-- Aligns primary friction with the x-axis (forward direction) -->
+                        <slip1>0.0</slip1>   <!-- Small slip value for slight sliding capability -->
+                        <slip2>0.0</slip2>   <!-- Small slip value for slight sliding capability -->
+                    </ode>
                 </friction>
             </surface>
@@ -238,11 +244,13 @@
     <gazebo reference="right_front_wheel">
         <material>Gazebo/Blue</material>
-        <!-- <kp>50000.0</kp>  -->
-        <!-- kp and kd for rubber -->
-        <!-- <kd>0.8</kd> -->
-        <mu1>1</mu1>
-        <mu2>1</mu2>
-        <maxVel>0.0</maxVel>
-        <minDepth>0.00005</minDepth>
+        <mu1>1.0</mu1>
+        <mu2>1.0</mu2>
+        <kp>1000000000000.0</kp>
+        <kd>10.0</kd>
+        <minDepth>0.0001</minDepth>
+        <maxVel>0.0</maxVel>
+        <fdir1>1 0 0</fdir1>
+        <slip1>0.0</slip1>   <!-- Small slip value for slight sliding capability -->
+        <slip2>0.0</slip2>
     </gazebo>
 </robot>

File: src/asitlorbot8_description/urdf/transmission.xacro (robot description, xacro)
@@ -2,24 +2,34 @@
 <robot xmlns:xacro="http://www.ros.org/wiki/xacro" >
     <!-- TRANSMISSION TAG INDICATES THE PRESENCE OF A MECHANCIAL TRANSMISSION THAT CONNECTS EACH MOTOR OF THE ROBOT TO EACH LINK OF THE LINK -->
-    <transmission name="joint_front_left_tran">
+    <transmission name="wheel_left_tran">
         <plugin>transmission_interface/SimpleTransmission</plugin>
-        <joint name="left_front_wheel_hinge">
-            <hardwareInterface>hardware_interface/VelocityJointInterface</hardwareInterface>
-        </joint>
-        <actuator name="joint_front_left_actr">
+        <actuator name="joint_front_left_actr" role="actuator_left">
             <hardwareInterface>hardware_interface/EffortJointInterface</hardwareInterface>
             <!-- 1 DEGREE OF ROTATION OF MOTOR CORRESPONDS TO 1 DEGREE OF ROTATION OF WHEEL -->
-            <mechanicalReduction>1</mechanicalReduction>
+            <mechanicalReduction>1.0</mechanicalReduction>
         </actuator>
+        <joint name="left_front_wheel_hinge" role="joint_left">
+            <hardwareInterface>hardware_interface/VelocityJointInterface</hardwareInterface>
+            <!-- <mechanical_reduction>1.0</mechanical_reduction> -->
+        </joint>
+        <joint name="left_back_wheel_hinge" role="joint_left">
+            <hardwareInterface>hardware_interface/VelocityJointInterface</hardwareInterface>
+            <!-- <mechanical_reduction>1.0</mechanical_reduction> -->
+        </joint>
     </transmission>
-    <transmission name="joint_front_right_tran">
+    <transmission name="wheel_right_tran">
         <plugin>transmission_interface/SimpleTransmission</plugin>
-        <joint name="right_front_wheel_hinge">
+        <actuator name="joint_front_right_actr" role="actuator_right">
+            <hardwareInterface>hardware_interface/EffortJointInterface</hardwareInterface>
+            <mechanicalReduction>1.0</mechanicalReduction>
+        </actuator>
+        <joint name="right_front_wheel_hinge" role="joint_right">
             <hardwareInterface>hardware_interface/VelocityJointInterface</hardwareInterface>
+            <!-- <mechanical_reduction>1.0</mechanical_reduction> -->
         </joint>
-        <actuator name="joint_front_right_actr">
-            <hardwareInterface>hardware_interface/EffortJointInterface</hardwareInterface>
-            <mechanicalReduction>1</mechanicalReduction>
-        </actuator>
+        <joint name="right_back_wheel_hinge" role="joint_right">
+            <hardwareInterface>hardware_interface/VelocityJointInterface</hardwareInterface>
+            <!-- <mechanical_reduction>1.0</mechanical_reduction> -->
+        </joint>
     </transmission>
     <!-- <transmission name="joint_rear_left_tran">
