Commit message: UPLOAD

File: src/asitlorbot8_description/urdf/robot_core.xacro (robot description, xacro)
@@ -65,5 +65,5 @@
         <axis xyz="0 0 1"/>
         <limit effort="10000.0" velocity="20.0" />
-        <dynamics damping="0"/>
+        <dynamics damping="0.0"/>
         <joint_properties friction="0.0" />
     </joint>
@@ -82,6 +82,6 @@
                 <friction>
                     <ode>
-                        <mu>10.0</mu>          <!-- Moderate grip in the primary direction -->
-                        <mu2>10.0</mu2>        <!-- Moderate grip in the secondary direction -->
+                        <mu>1.0</mu>          <!-- Moderate grip in the primary direction -->
+                        <mu2>1.0</mu2>        <!-- Moderate grip in the secondary direction -->
                         <fdir1>1 0 0</fdir1>  <!-- Aligns primary friction with the x-axis (forward direction) -->
                         <slip1>0.0</slip1>   <!-- Small slip value for slight sliding capability -->
@@ -114,5 +114,5 @@
         <axis xyz="0 0 1"/>
         <limit effort="10000.0" velocity="20.0" />
-        <dynamics damping="0"/>
+        <dynamics damping="0.0"/>
         <joint_properties friction="0.0" />
     </joint>
@@ -163,5 +163,5 @@
         <axis xyz="0 0 -1"/>
         <limit effort="10000.0" velocity="20.0" />
-        <dynamics damping="0"/>
+        <dynamics damping="0.0"/>
         <joint_properties friction="0.0" />
     </joint>
@@ -212,5 +212,5 @@
         <axis xyz="0 0 -1"/>
         <limit effort="10000.0" velocity="20.0" />
-        <dynamics damping="0"/>
+        <dynamics damping="0.0"/>
         <joint_properties friction="0.0" />
     </joint>
